File: cad/temp-sensor(v1).brd (EAGLE design)
At the start: 100 x 80 mm, 47 parts, among them Q1 300S14-U, Q2 320S14-U, Q3 320S14-U, U1 SE555D, U2 SE555D, U4 MCP6001UT-I/OT, U5 MCP6001UT-I/OT, U6 MCP6001UT-I/OT, U7 MCP6001UT-I/OT, U8 NCV4264-2CST50T3G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

Commit message: Add files via upload
Both board files are preliminary layouts. Not all components are present. temp-sensor(v1) was my first pass of beginning the layout.
Parts:
- moved R3 141.7 mm to (77.3, 47.5), turned to 90 degrees
- moved C3 138.8 mm to (79.4, 43.6), turned to 90 degrees
- moved C6 138.3 mm to (65.3, 33.8), turned to 270 degrees
- moved R7 137.5 mm to (52.5, 30.5)
- moved C7 137.1 mm to (63.2, 48.1), turned to 90 degrees
- moved R4 135.9 mm to (64.8, 37.5), turned to 180 degrees
- moved R5 134.7 mm to (56.5, 28.8), turned to 270 degrees
- moved R6 131.9 mm to (55.6, 46.7)
- moved C8 130.0 mm to (52.2, 48.0), turned to 90 degrees
- moved R2 124.5 mm to (65.0, 54.6), turned to 270 degrees
- moved R1 122.4 mm to (65.8, 51.0), turned to 180 degrees
- moved C5 122.3 mm to (54.5, 41.3)
- moved C4 113.9 mm to (50.2, 43.9), turned to 180 degrees
- moved R8 107.6 mm to (81.8, 36.0)
- moved C14 100.1 mm to (57.2, 38.3), turned to 270 degrees
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