File: cad/temp-sensor.sch (EAGLE design)
At the start: 31 parts, among them IC1 320S14-U, IC2 320S14-U, Q1 300S14-U, U1 SE555D, U2 SE555D

Commit message: Add MCU and LDO, Initialize .BRD file
Parts:
- removed OPAMP1, OPAMP2, OPAMP3, OPAMP4: MCP6001UT-I/OT, MCP600:MCP6001UT-I/OT
- added C11, C12, C13, C14: 10nF, SparkFun-Capacitors:10NF-0603-50V-10%
- added C15, C16: 10uF, SparkFun-Capacitors:10UF-0805-25V-10%
- added C17, C18: 0.1uF, SparkFun-Capacitors:0.1UF-0603-25V-10%-X7R-WE
- added C19, C20: 18pF, SparkFun-Capacitors:18PF-0603-50V-5%
- added R13: 0, SparkFun-Resistors:0OHM-0603-1/10W
- added R14, R15: 5.1k, SparkFun-Resistors:5.1KOHM5.1KOHM-0603-1/10W-1%
- added R16: 100k, SparkFun-Resistors:100KOHM-0603-1/10W-1%
- added U4, U5, U6, U7: MCP6001UT-I/OT, MCP6001UT-I_OT:MCP6001UT-I/OT
- added U8: NCV4264-2CST50T3G, NCV4264-2CST50T3G:NCV4264-2CST50T3G
- added U9: ATMEGA328P_TQFP, SparkFun-IC-Microcontroller:ATMEGA328P_TQFP
- R3: value 1k -> 1.8k; device SparkFun-Resistors:1KOHM-0603-1/10W-1% -> SparkFun-Resistors:1.8KOHM-0603-1/10W-1%
- R5: value 100k -> 200k; device SparkFun-Resistors:100KOHM-0603-1/10W-1% -> SparkFun-Resistors:200KOHM-0603-1/10W-1%
- R6: value 100k -> 0; device SparkFun-Resistors:100KOHM-0603-1/10W-1% -> SparkFun-Resistors:0OHM-0603-1/10W
- R8: value 1k -> 100; device SparkFun-Resistors:1KOHM-0603-1/10W-1% -> SparkFun-Resistors:100OHM-0603-1/10W-1%
- renumbered IC1 to Q3, IC2 to Q2
Connections:
- removed net BG_REF_FD_BK: OPAMP2.VIN-, R4.1, R6.2
- removed net N$1: R5.2, R6.1
- removed net N$11: C4.2, U1.GND
- removed net N$12: U2.GND
- removed net N$2: Q2.E3
- removed net N$3: Q2.E1
- new net +9V: U8.VIN
- new net BG_REF_FB: C11.1, R4.1, R5.2, U5.VIN-
- new net CIPO: U9.PB4(CIPO)
- new net COPI: U9.PB3(COPI/OC2)
- new net MCU_RST: R16.1, U9.PC6(/RESET)
- new net N$7: U1.RESET
- new net N$8: U1.DISCH
- new net N$9: U2.RESET
- new net PTAT_REF_FB: C13.1, R13.1, R6.2, U7.VIN-
- new net SCK: U9.PB5(SCK)
- new net SCL: R15.1, U9.PC5(ADC5/SCL)
- new net SDA: R14.1, U9.PC4(ADC4/SDA)
- new net SS: U9.PB2(SS/OC1B)
- net +5V: now also C15.1, C16.1, C17.1, C18.1, Q2.E1, Q2.E2, Q2.E3, Q2.E4, R14.2, R15.2, R16.2, R2.2, U4.VDD, U5.VDD, U6.VDD, U7.VDD, U8.VOUT, U9.AVCC, U9.VCC; no longer OPAMP1.VDD, OPAMP2.VDD, OPAMP3.VDD, OPAMP4.VDD, R3.2, U1.RESET, U2.RESET
- net CTAT_BASE: now also U4.VOUT; no longer OPAMP1.VOUT
- net CTAT_E1: now also R2.1; no longer R3.1
- net CTAT_IN+: now also R3.2, U4.VIN+; no longer OPAMP1.VIN+, R2.2
- net GND: now also C11.2, C12.2, C13.2, C14.2, C15.2, C16.2, C17.2, C18.2, C19.1, C20.1, C4.2, R3.1, R6.1, U1.GND, U2.GND, U4.VSS, U5.VSS, U6.VSS, U7.VSS, U8.EPAD, U8.GND, U9.AGND, U9.GND; no longer OPAMP1.VSS, OPAMP2.VSS, OPAMP3.VSS, OPAMP4.VSS, R2.1
- net I_BG: now also C12.1, U5.VIN+; no longer OPAMP2.VIN+
- net I_PTAT: now also C14.1, U7.VIN+; no longer OPAMP4.VIN+
- net N$4: now also C19.2, U9.PB6(XTAL1/TOSC1); no longer Q2.E4
- net N$5: now also C20.2, U9.PB7(XTAL2/TOSC2); no longer Q2.E2
- net PTAT_BASE: now also U6.VOUT; no longer OPAMP3.VOUT
- net PTAT_IN+: now also U6.VIN+; no longer OPAMP3.VIN+
- net PULSE_THRES: no longer U1.DISCH
- net TEMP_VBE: now also U4.VIN-, U6.VIN-; no longer OPAMP1.VIN-, OPAMP3.VIN-
- net VBG_REF: now also U5.VOUT; no longer OPAMP2.VOUT
- net VPTAT_REF: now also R13.2, U7.VOUT; no longer OPAMP4.VIN-, OPAMP4.VOUT
Other:
- note added: "Battery connection"
- note added: "DO NOT POPULATE R6"
- note added: "LDO Voltage Regulator"
- note added: "May not need to populate C11, C12"
- note added: "May not need to populate C13, C14"
- note added: "U1 is in monostable mode"
- note added: "U2 is in astable mode"
- note removed: "U1 will be our monostable timer"
- moved on the sheet: C5, R11, R2, R3, R5, R6
