File: cad/temp-sensor.brd (EAGLE design)
At the start: 172.5 x 41 mm, 61 parts, among them Q1 300S14-U, Q2 320S14-U, Q3 320S14-U, U1 SE555D, U2 SE555D, U4 MCP6001UT-I/OT, U6 MCP6001UT-I/OT, U7 MCP6001UT-I/OT, U8 NCV4264-2CST50T3G, U9 ATMEGA328P_TQFP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

Commit message: Adjust grid and via placement
Parts:
- moved R22 1.80 mm to (30.5, 20.3)
Routing:
- net TEMP_VBE: track 71.9 -> 77.0 mm
- net GND: track 107.7 -> 110.9 mm
- net START_C: track 27.5 -> 25.6 mm
- net CTAT_BASE: track 23.8 -> 22.0 mm
- net CTAT_IN+: track 15.4 -> 16.9 mm
- net PTAT_IN+: track 31.7 -> 33.0 mm
- net I_BG: track 47.3 -> 46.3 mm
- net PTAT_BASE: track 70.9 -> 71.6 mm
